Commit message: ros2 control update

File: src/ant_description/urdf/ant.ros2_control.xacro (robot description, xacro)
@@ -8,5 +8,8 @@
             </hardware>
             <joint name="joint1Leg">
-                <command_interface name="effort"/>
+            <command_interface name="position">
+                <param name="min">-1.570796</param>
+                <param name="max">1.570796</param>
+            </command_interface>
                 <state_interface name="position">
                   <param name="initial_value">${initial_positions['joint1Leg']}</param>
@@ -16,5 +19,8 @@
             </joint>
             <joint name="joint2Leg">
-                <command_interface name="effort"/>
+            <command_interface name="position">
+                <param name="min">-1.570796</param>
+                <param name="max">1.570796</param>
+            </command_interface>
                 <state_interface name="position">
                   <param name="initial_value">${initial_positions['joint2Leg']}</param>
@@ -24,5 +30,8 @@
             </joint>
             <joint name="joint3Leg">
-                <command_interface name="effort"/>
+            <command_interface name="position">
+                <param name="min">-1.570796</param>
+                <param name="max">1.570796</param>
+            </command_interface>
                 <state_interface name="position">
                   <param name="initial_value">${initial_positions['joint3Leg']}</param>
@@ -32,5 +41,8 @@
             </joint>
             <joint name="joint1Leg_2">
-                <command_interface name="effort"/>
+            <command_interface name="position">
+                <param name="min">-1.570796</param>
+                <param name="max">1.570796</param>
+            </command_interface>
                 <state_interface name="position">
                   <param name="initial_value">${initial_positions['joint1Leg_2']}</param>
@@ -40,5 +52,8 @@
             </joint>
             <joint name="joint2Leg_2">
-                <command_interface name="effort"/>
+            <command_interface name="position">
+                <param name="min">-1.570796</param>
+                <param name="max">1.570796</param>
+            </command_interface>
                 <state_interface name="position">
                   <param name="initial_value">${initial_positions['joint2Leg_2']}</param>
@@ -48,5 +63,8 @@
             </joint>
             <joint name="joint3Leg_2">
-                <command_interface name="effort"/>
+            <command_interface name="position">
+                <param name="min">-1.570796</param>
+                <param name="max">1.570796</param>
+            </command_interface>
                 <state_interface name="position">
                   <param name="initial_value">${initial_positions['joint3Leg_2']}</param>
@@ -56,5 +74,8 @@
             </joint>
             <joint name="joint1Leg_3">
-                <command_interface name="effort"/>
+            <command_interface name="position">
+                <param name="min">-1.570796</param>
+                <param name="max">1.570796</param>
+            </command_interface>
                 <state_interface name="position">
                   <param name="initial_value">${initial_positions['joint1Leg_3']}</param>
@@ -64,5 +85,8 @@
             </joint>
             <joint name="joint2Leg_3">
-                <command_interface name="effort"/>
+            <command_interface name="position">
+                <param name="min">-1.570796</param>
+                <param name="max">1.570796</param>
+            </command_interface>
                 <state_interface name="position">
                   <param name="initial_value">${initial_positions['joint2Leg_3']}</param>
@@ -72,5 +96,8 @@
             </joint>
             <joint name="joint3Leg_3">
-                <command_interface name="effort"/>
+            <command_interface name="position">
+                <param name="min">-1.570796</param>
+                <param name="max">1.570796</param>
+            </command_interface>
                 <state_interface name="position">
                   <param name="initial_value">${initial_positions['joint3Leg_3']}</param>
@@ -80,5 +107,8 @@
             </joint>
             <joint name="joint1Leg_4">
-                <command_interface name="effort"/>
+            <command_interface name="position">
+                <param name="min">-1.570796</param>
+                <param name="max">1.570796</param>
+            </command_interface>
                 <state_interface name="position">
                   <param name="initial_value">${initial_positions['joint1Leg_4']}</param>
@@ -88,5 +118,8 @@
             </joint>
             <joint name="joint2Leg_4">
-                <command_interface name="effort"/>
+            <command_interface name="position">
+                <param name="min">-1.570796</param>
+                <param name="max">1.570796</param>
+            </command_interface>
                 <state_interface name="position">
                   <param name="initial_value">${initial_positions['joint2Leg_4']}</param>
@@ -96,5 +129,8 @@
             </joint>
             <joint name="joint3Leg_4">
-                <command_interface name="effort"/>
+            <command_interface name="position">
+                <param name="min">-1.570796</param>
+                <param name="max">1.570796</param>
+            </command_interface>
                 <state_interface name="position">
                   <param name="initial_value">${initial_positions['joint3Leg_4']}</param>
@@ -104,5 +140,8 @@
             </joint>
             <joint name="joint1Leg_5">
-                <command_interface name="effort"/>
+            <command_interface name="position">
+                <param name="min">-1.570796</param>
+                <param name="max">1.570796</param>
+            </command_interface>
                 <state_interface name="position">
                   <param name="initial_value">${initial_positions['joint1Leg_5']}</param>
@@ -112,5 +151,8 @@
             </joint>
             <joint name="joint2Leg_5">
-                <command_interface name="effort"/>
+             <command_interface name="position">
+                <param name="min">-1.570796</param>
+                <param name="max">1.570796</param>
+            </command_interface>
                 <state_interface name="position">
                   <param name="initial_value">${initial_positions['joint2Leg_5']}</param>
@@ -120,5 +162,8 @@
             </joint>
             <joint name="joint3Leg_5">
-                <command_interface name="effort"/>
+            <command_interface name="position">
+                <param name="min">-1.570796</param>
+                <param name="max">1.570796</param>
+            </command_interface>
                 <state_interface name="position">
                   <param name="initial_value">${initial_positions['joint3Leg_5']}</param>
@@ -128,5 +173,8 @@
             </joint>
             <joint name="joint1Leg_6">
-                <command_interface name="effort"/>
+            <command_interface name="position">
+                <param name="min">-1.570796</param>
+                <param name="max">1.570796</param>
+            </command_interface>
                 <state_interface name="position">
                   <param name="initial_value">${initial_positions['joint1Leg_6']}</param>
@@ -136,5 +184,8 @@
             </joint>
             <joint name="joint2Leg_6">
-                <command_interface name="effort"/>
+            <command_interface name="position">
+                <param name="min">-1.570796</param>
+                <param name="max">1.570796</param>
+            </command_interface>
                 <state_interface name="position">
                   <param name="initial_value">${initial_positions['joint2Leg_6']}</param>
@@ -144,5 +195,8 @@
             </joint>
             <joint name="joint3Leg_6">
-                <command_interface name="effort"/>
+            <command_interface name="position">
+                <param name="min">-1.570796</param>
+                <param name="max">1.570796</param>
+            </command_interface>
                 <state_interface name="position">
                   <param name="initial_value">${initial_positions['joint3Leg_6']}</param>
@@ -150,4 +204,22 @@
                 <state_interface name="velocity"/>
                 <state_interface name="effort"/>
+            </joint>
+            <joint name = "rightJawJoint">
+             <command_interface name="position">
+                <param name="min">-1.5707960796</param>
+                <param name="max">0.06</param>
+            </command_interface>
+            <state_interface name="position">
+                  <param name="initial_value">0.0</param>
+            </state_interface>
+            <state_interface name="velocity"/>
+            </joint>
+            <joint name = "leftJawJoint">
+              <param name = "mimic">rightJawJoint</param>
+              <param name="multiplier">1</param>
+            <state_interface name="position">
+                  <param name="initial_value">0.0</param>
+            </state_interface>
+            <state_interface name="velocity"/>
             </joint>
         </ros2_control>
