Commit message: added controller launch file

File: src/ant_description/urdf/ant.core.xacro (robot description, xacro)
@@ -1,4 +1,10 @@
 <?xml version="1.0"?>
 <robot xmlns:xacro="http://www.ros.org/wiki/xacro" name="ant_robot_body">
+    <!-- <link name="world"/>
+    <joint name="world_to_robot_base" type="fixed">
+        <parent link="world"/>
+        <child link="robot_base"/>
+        <origin xyz="0 0 0" rpy="0 0 0"/>
+    </joint> -->
     <link name="robot_base">
         <inertial>
