Commit message: Initial commit

File: src/hexapod_description/urdf/hexapod.core.xacro (robot description, xacro)
@@ -35,9 +35,10 @@
         </visual>
     </link>
-    <joint type="continuous" name="joint1_">
+    <joint type="revolute" name="joint1_">
         <axis xyz="0 0 1" />
         <parent link="robot_base" />
         <child link="link1Respondable_" />
         <origin rpy="3.141593 3.141593 3.141593" xyz="0.080000 -0.000000 0.091002" />
+        <limit lower="-1.570796" upper="1.570796" effort="5" velocity="2"/>
     </joint>
     <link name="link1Respondable_">
@@ -84,9 +85,10 @@
         </visual>
     </link>
-    <joint type="continuous" name="joint2_">
+    <joint type="revolute" name="joint2_">
         <axis xyz="0 0 1" />
         <parent link="link1Respondable_" />
         <child link="link2Respondable_" />
         <origin rpy="1.570796 3.141593 3.141593" xyz="0.050264 -0.000000 -0.011203" />
+        <limit lower="-1.570796" upper="1.570796" effort="5" velocity="2"/>
     </joint>
     <link name="link2Respondable_">
@@ -139,9 +141,10 @@
         </visual>
     </link>
-    <joint type="continuous" name="joint3_">
+    <joint type="revolute" name="joint3_">
         <axis xyz="0 0 1" />
         <parent link="link2Respondable_" />
         <child link="link3Respondable_" />
         <origin rpy="-3.141593 3.141593 -2.617994" xyz="0.072382 0.000000 -0.000000" />
+        <limit lower="-1.570796" upper="1.570796" effort="5" velocity="2"/>
     </joint>
     <link name="link3Respondable_">
@@ -218,9 +221,10 @@
         </visual>
     </link>
-    <joint type="continuous" name="joint1__2">
+    <joint type="revolute" name="joint1__2">
         <axis xyz="0 0 1" />
         <parent link="robot_base" />
         <child link="link1Respondable__2" />
         <origin rpy="3.141592 3.141593 -2.094395" xyz="0.040000 0.069282 0.091002" />
+        <limit lower="-1.570796" upper="1.570796" effort="5" velocity="2"/>
     </joint>
     <link name="link1Respondable__2">
@@ -267,9 +271,10 @@
         </visual>
     </link>
-    <joint type="continuous" name="joint2__2">
+    <joint type="revolute" name="joint2__2">
         <axis xyz="0 0 1" />
         <parent link="link1Respondable__2" />
         <child link="link2Respondable__2" />
         <origin rpy="1.570796 3.141593 3.141593" xyz="0.050264 -0.000000 -0.011203" />
+        <limit lower="-1.570796" upper="1.570796" effort="5" velocity="2"/>
     </joint>
     <link name="link2Respondable__2">
@@ -322,9 +327,10 @@
         </visual>
     </link>
-    <joint type="continuous" name="joint3__2">
+    <joint type="revolute" name="joint3__2">
         <axis xyz="0 0 1" />
         <parent link="link2Respondable__2" />
         <child link="link3Respondable__2" />
         <origin rpy="-3.141593 3.141593 -2.617994" xyz="0.072382 0.000000 -0.000000" />
+        <limit lower="-1.570796" upper="1.570796" effort="5" velocity="2"/>
     </joint>
     <link name="link3Respondable__2">
@@ -401,9 +407,10 @@
         </visual>
     </link>
-    <joint type="continuous" name="joint1__3">
+    <joint type="revolute" name="joint1__3">
         <axis xyz="0 0 1" />
         <parent link="robot_base" />
         <child link="link1Respondable__3" />
         <origin rpy="3.141592 3.141593 -1.047197" xyz="-0.040000 0.069282 0.091002" />
+        <limit lower="-1.570796" upper="1.570796" effort="5" velocity="2"/>
     </joint>
     <link name="link1Respondable__3">
@@ -450,9 +457,10 @@
         </visual>
     </link>
-    <joint type="continuous" name="joint2__3">
+    <joint type="revolute" name="joint2__3">
         <axis xyz="0 0 1" />
         <parent link="link1Respondable__3" />
         <child link="link2Respondable__3" />
         <origin rpy="1.570796 3.141593 3.141593" xyz="0.050264 -0.000000 -0.011203" />
+        <limit lower="-1.570796" upper="1.570796" effort="5" velocity="2"/>
     </joint>
     <link name="link2Respondable__3">
@@ -505,9 +513,10 @@
         </visual>
     </link>
-    <joint type="continuous" name="joint3__3">
+    <joint type="revolute" name="joint3__3">
         <axis xyz="0 0 1" />
         <parent link="link2Respondable__3" />
         <child link="link3Respondable__3" />
         <origin rpy="-3.141593 3.141593 -2.617994" xyz="0.072382 0.000000 -0.000000" />
+        <limit lower="-1.570796" upper="1.570796" effort="5" velocity="2"/>
     </joint>
     <link name="link3Respondable__3">
@@ -584,9 +593,10 @@
         </visual>
     </link>
-    <joint type="continuous" name="joint1__4">
+    <joint type="revolute" name="joint1__4">
         <axis xyz="0 0 1" />
         <parent link="robot_base" />
         <child link="link1Respondable__4" />
         <origin rpy="-3.141593 3.141592 0.000000" xyz="-0.080000 0.000000 0.091002" />
+        <limit lower="-1.570796" upper="1.570796" effort="5" velocity="2"/>
     </joint>
     <link name="link1Respondable__4">
@@ -633,9 +643,10 @@
         </visual>
     </link>
-    <joint type="continuous" name="joint2__4">
+    <joint type="revolute" name="joint2__4">
         <axis xyz="0 0 1" />
         <parent link="link1Respondable__4" />
         <child link="link2Respondable__4" />
         <origin rpy="1.570796 3.141593 -3.141593" xyz="0.050264 -0.000000 -0.011203" />
+        <limit lower="-1.570796" upper="1.570796" effort="5" velocity="2"/>
     </joint>
     <link name="link2Respondable__4">
@@ -688,9 +699,10 @@
         </visual>
     </link>
-    <joint type="continuous" name="joint3__4">
+    <joint type="revolute" name="joint3__4">
         <axis xyz="0 0 1" />
         <parent link="link2Respondable__4" />
         <child link="link3Respondable__4" />
         <origin rpy="-3.141593 3.141593 -2.617994" xyz="0.072382 0.000000 -0.000000" />
+        <limit lower="-1.570796" upper="1.570796" effort="5" velocity="2"/>
     </joint>
     <link name="link3Respondable__4">
@@ -767,9 +779,10 @@
         </visual>
     </link>
-    <joint type="continuous" name="joint1__5">
+    <joint type="revolute" name="joint1__5">
         <axis xyz="0 0 1" />
         <parent link="robot_base" />
         <child link="link1Respondable__5" />
         <origin rpy="-3.141592 3.141593 1.047198" xyz="-0.040000 -0.069282 0.091002" />
+        <limit lower="-1.570796" upper="1.570796" effort="5" velocity="2"/>
     </joint>
     <link name="link1Respondable__5">
@@ -816,9 +829,10 @@
         </visual>
     </link>
-    <joint type="continuous" name="joint2__5">
+    <joint type="revolute" name="joint2__5">
         <axis xyz="0 0 1" />
         <parent link="link1Respondable__5" />
         <child link="link2Respondable__5" />
         <origin rpy="1.570796 3.141593 -3.141593" xyz="0.050264 -0.000000 -0.011203" />
+        <limit lower="-1.570796" upper="1.570796" effort="5" velocity="2"/>
     </joint>
     <link name="link2Respondable__5">
@@ -871,9 +885,10 @@
         </visual>
     </link>
-    <joint type="continuous" name="joint3__5">
+    <joint type="revolute" name="joint3__5">
         <axis xyz="0 0 1" />
         <parent link="link2Respondable__5" />
         <child link="link3Respondable__5" />
         <origin rpy="-3.141593 3.141593 -2.617994" xyz="0.072382 0.000000 -0.000000" />
+        <limit lower="-1.570796" upper="1.570796" effort="5" velocity="2"/>
     </joint>
     <link name="link3Respondable__5">
@@ -950,9 +965,10 @@
         </visual>
     </link>
-    <joint type="continuous" name="joint1__6">
+    <joint type="revolute" name="joint1__6">
         <axis xyz="0 0 1" />
         <parent link="robot_base" />
         <child link="link1Respondable__6" />
         <origin rpy="-3.141592 3.141593 2.094395" xyz="0.040000 -0.069282 0.091002" />
+        <limit lower="-1.570796" upper="1.570796" effort="5" velocity="2"/>
     </joint>
     <link name="link1Respondable__6">
@@ -999,9 +1015,10 @@
         </visual>
     </link>
-    <joint type="continuous" name="joint2__6">
+    <joint type="revolute" name="joint2__6">
         <axis xyz="0 0 1" />
         <parent link="link1Respondable__6" />
         <child link="link2Respondable__6" />
         <origin rpy="1.570796 3.141593 -3.141593" xyz="0.050264 -0.000000 -0.011203" />
+        <limit lower="-1.570796" upper="1.570796" effort="5" velocity="2"/>
     </joint>
     <link name="link2Respondable__6">
@@ -1054,9 +1071,10 @@
         </visual>
     </link>
-    <joint type="continuous" name="joint3__6">
+    <joint type="revolute" name="joint3__6">
         <axis xyz="0 0 1" />
         <parent link="link2Respondable__6" />
         <child link="link3Respondable__6" />
         <origin rpy="-3.141593 3.141593 -2.617994" xyz="0.072382 0.000000 -0.000000" />
+        <limit lower="-1.570796" upper="1.570796" effort="5" velocity="2"/>
     </joint>
     <link name="link3Respondable__6">
